Commit message: added final project with modified code for policy evaluator and features

File: ros_ws/src/franka_ros/panda_moveit_config/config/panda_arm.xacro (robot description, xacro)
@@ -13,5 +13,5 @@
     <group_state name="ready" group="panda_arm">
       <joint name="panda_joint1" value="0" />
-      <joint name="panda_joint2" value="-1.0472" />
+      <joint name="panda_joint2" value="-0.785" />
       <joint name="panda_joint3" value="0" />
       <joint name="panda_joint4" value="-2.356" />

File: ros_ws/src/projects/active_vision/desc/franka_camera.xacro (robot description, xacro)
@@ -3,5 +3,5 @@
 <robot xmlns:xacro="http://www.ros.org/wiki/xacro" name="panda_hand_camera">
   <!-- Include xacro files -->
-  <xacro:include filename="$(find franka_description)/robots/panda_arm_hand_active_vision.xacro"/>
+  <xacro:include filename="/home/uthira/mer_lab/ros_ws/src/desc/franka_description/robots/panda_arm_hand_active_vision.xacro"/>
   <xacro:include filename="$(find active_vision)/desc/depth.xacro" />
   <link name="end_effector_link" />
